Commit message: Add a first-attempt at having the robot play an actual song

File: theremini_description/urdf/theremini.urdf.xacro (robot description, xacro)
@@ -74,5 +74,5 @@
       <parent link="${prefix}_body" />
       <child link="${prefix}_pitch_antenna" />
-      <origin xyz="0 -0.22 0.01" rpy="0 0 0" />
+      <origin xyz="0 -0.22 0.01" rpy="0 0 ${pi}" />
     </joint>
     <link name="${prefix}_volume_antenna">
